File: flashlight_solder.kicad_sch (KiCad schematic)
At the start: 6 parts, among them SW1 SW_Push

Commit message: Change to different battery holder part
- lower profile
- battery less likely to fall out
Parts:
- BT1: footprint fl-parts:CR2032-THT -> fl-parts:CR2032-THT-retainer
Changed lines of the file:
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@@
 			)
 		)
-		(property "Footprint" "fl-parts:CR2032-THT"
+		(property "Footprint" "fl-parts:CR2032-THT-retainer"
 			(at 73.66 72.136 90)
 			(effects
