File: var-tone-beeper/var-tone-beeper.kicad_sch (KiCad schematic)
At the start: 10 parts, among them SW1 SW_Push, U1 NE555P

Commit message: var-tone-beeper bugfixes
fixed schematics bug
switched to 23mm speaker only
made proper footprint for batttery box
Parts:
- BT1: value Battery_Cell -> 3xAAA; footprint Battery:BatteryHolder_MPD_BC2AAPC_2xAA -> fl-parts:BatteryHolder_Generic_3xAAA
- LS1: footprint fl-parts:PC-mnt-speaker-23-30-mm -> fl-parts:PC-mnt-speaker-23-mm
Connections:
- net at U1.2 (TR), U1.6 (THR): now also C1.1, C2.1, JP1.2 (C)
- net at R2.1, SW1.2, U1.4 (R)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: no longer C1.1, C2.1, JP1.2 (C)
Changed lines of the file:
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@@
 	(paper "A4")
-	(junction
-		(at 144.78 80.01)
-		(diameter 0)
-		(color 0 0 0 0)
-	)
 	(junction
 		(at 138.43 66.04)
@@
 	)
 	(junction
+		(at 149.86 85.09)
+		(diameter 0)
+		(color 0 0 0 0)
+	)
+	(junction
 		(at 124.46 58.42)
 		(diameter 0)
@@
 	(wire
 		(pts
-			(xy 144.78 80.01) (xy 144.78 85.09)
-		)
-		(stroke
-			(width 0)
-			(type default)
-		)
-	)
-	(wire
-		(pts
 			(xy 123.19 74.93) (xy 123.19 80.01)
 		)
@@
 	(wire
 		(pts
+			(xy 149.86 85.09) (xy 149.86 88.9)
+		)
+		(stroke
+			(width 0)
+			(type default)
+		)
+	)
+	(wire
+		(pts
 			(xy 156.21 80.01) (xy 144.78 80.01)
 		)
@@
 	(wire
 		(pts
-			(xy 118.11 85.09) (xy 144.78 85.09)
+			(xy 118.11 85.09) (xy 149.86 85.09)
 		)
 		(stroke
@@
 	(wire
 		(pts
-			(xy 149.86 69.85) (xy 149.86 88.9)
+			(xy 149.86 69.85) (xy 149.86 85.09)
 		)
 		(stroke
@@
 			)
 		)
-		(property "Value" "Battery_Cell"
+		(property "Value" "3xAAA"
 			(at 91.44 73.0884 0)
 			(effects
@@
 			)
 		)
-		(property "Footprint" "Battery:BatteryHolder_MPD_BC2AAPC_2xAA"
+		(property "Footprint" "fl-parts:BatteryHolder_Generic_3xAAA"
 			(at 87.63 72.136 90)
 			(effects
@@
 			)
 		)
-		(property "Footprint" "fl-parts:PC-mnt-speaker-23-30-mm"
+		(property "Footprint" "fl-parts:PC-mnt-speaker-23-mm"
 			(at 196.85 74.93 0)
 			(effects

Commit message: ver-tone-beeper: v1 ordered
Reduced board size
Ordered

JLCPCB cost: 10x for $14.10 + $8.36 shipping/tax
Parts:
- JP1: footprint Jumper:SolderJumper-3_P1.3mm_Bridged2Bar12_RoundedPad1.0x1.5mm -> Jumper:SolderJumper-3_P1.3mm_Bridged12_RoundedPad1.0x1.5mm
Changed lines of the file:
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@@
 			)
 		)
-		(property "Footprint" "Jumper:SolderJumper-3_P1.3mm_Bridged2Bar12_RoundedPad1.0x1.5mm"
+		(property "Footprint" "Jumper:SolderJumper-3_P1.3mm_Bridged12_RoundedPad1.0x1.5mm"
 			(at 118.11 80.01 0)
 			(effects
