File: led-letter-5x7/led-letter-5x7.kicad_pcb (KiCad board)
At the start: 2 copper layers, 33 x 53.3 mm, 20 parts, among them J1 PROG, J2 POWER (TODO CHECK POL), SW1 SW_SPDT, SW2 SELECT, SW3 INC, SW4 DEC, U1 STC8G1K08-38I-DIP16

Commit message: led-letter-5x7: v1 done, ordered
Moved battery to the bottom
Make outline more interesting

Added README with parts list
Parts:
- BT1: moved to F.Cu
- moved BT1 38.2 mm to (142.2, 135.9)
- moved G*** 24.0 mm to (145.4, 90.8)
- moved J2 0.57 mm to (134.1, 81.8)
Routing:
- net Net-(BT1-+): track 22.4 -> 60.7 mm
- net GND: track 109.4 -> 111.2 mm
Other:
- board size 33 x 53.3 mm -> 33 x 79.4 mm
- board text added: "+"
- board text added: "-"
- board text added: "Assembled by:"
