File: led-letter-5x7/led-letter-5x7.kicad_sch (KiCad schematic)
At the start: 19 parts, among them J1 PROG, J2 POWER (TODO CHECK POL), SW1 SW_SPDT, SW2 SELECT, SW3 INC, SW4 DEC, U1 STC8G1K08-38I-DIP16

Commit message: led-letter-5x7: v1 done, ordered
Moved battery to the bottom
Make outline more interesting

Added README with parts list
Parts:
- J2: value POWER (TODO CHECK POL) -> POWER
Changed lines of the file:
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@@
 			)
 		)
-		(property "Value" "POWER (TODO CHECK POL)"
+		(property "Value" "POWER"
 			(at 36.195 82.55 0)
 			(effects
